File: rs485-usb.sch (KiCad schematic (older format))
At the start: 14 parts, among them J1 RJ45, P1 USBMICRO, P2 CONN_6, P3 CONN_6, P4 CONN_6, P5 CONN_2, U1 FT232RL, U2 MAX488

Commit message: Created first pass at board
Parts:
- removed P3: CONN_6, symbol CONN_6
- added LED3: PWR, ~, symbol LED
- added R4: 1k, ~, symbol R
- P2: value CONN_6 -> FTDI
- P3: renamed from P4; value CONN_6 -> FTDI
Connections:
- net +5V: now also R4.1
- net GND: now also U1.18 (GND), U1.25 (AGND), U1.26 (TEST), U1.7 (GND), LED3.2 (K)
- new net: LED3.1 (A), R4.2
Changed lines of the file:
@@
 P 5050 4500
 F 0 "P2" V 5000 4500 60  0000 C CNN
-F 1 "CONN_6" V 5100 4500 60  0000 C CNN
+F 1 "FTDI" V 5100 4500 60  0000 C CNN
 F 2 "" H 5050 4500 60  0000 C CNN
 F 3 "" H 5050 4500 60  0000 C CNN
@@
 	2250 1600 2400 1600
 Connection ~ 2250 1500
-Wire Wire Line
-	3050 3450 3650 3450
 Connection ~ 3200 3450
 Connection ~ 3350 3450
-Wire Wire Line
-	3500 3450 3500 3500
-$Comp
-L GND #PWR06
-U 1 1 528AE2E8
-P 3500 3500
-F 0 "#PWR06" H 3500 3500 30  0001 C CNN
-F 1 "GND" H 3500 3430 30  0001 C CNN
-F 2 "" H 3500 3500 60  0000 C CNN
-F 3 "" H 3500 3500 60  0000 C CNN
-	1    3500 3500
-	1    0    0    -1
-$EndComp
 NoConn ~ 2400 2250
 NoConn ~ 2400 2450
@@
 	1700 1950 2400 1950
 $Comp
-L GND #PWR07
+L GND #PWR06
 U 1 1 528AE2C6
 P 1900 2250
-F 0 "#PWR07" H 1900 2250 30  0001 C CNN
+F 0 "#PWR06" H 1900 2250 30  0001 C CNN
 F 1 "GND" H 1900 2180 30  0001 C CNN
 F 2 "" H 1900 2250 60  0000 C CNN
@@
 	1900 2150 1900 2250
 $Comp
-L +5V #PWR08
+L +5V #PWR07
 U 1 1 528AE2FF
 P 1850 1600
-F 0 "#PWR08" H 1850 1690 20  0001 C CNN
+F 0 "#PWR07" H 1850 1690 20  0001 C CNN
 F 1 "+5V" H 1850 1690 30  0000 C CNN
 F 2 "" H 1850 1600 60  0000 C CNN
@@
 	1700 2050 1700 2150
 $Comp
-L GND #PWR09
+L GND #PWR08
 U 1 1 528AE444
 P 8450 2400
-F 0 "#PWR09" H 8450 2400 30  0001 C CNN
+F 0 "#PWR08" H 8450 2400 30  0001 C CNN
 F 1 "GND" H 8450 2330 30  0001 C CNN
 F 2 "" H 8450 2400 60  0000 C CNN
@@
 $EndComp
 $Comp
-L +5V #PWR010
+L +5V #PWR09
 U 1 1 528AE48D
 P 1700 2550
-F 0 "#PWR010" H 1700 2640 20  0001 C CNN
+F 0 "#PWR09" H 1700 2640 20  0001 C CNN
 F 1 "+5V" H 1700 2640 30  0000 C CNN
 F 2 "" H 1700 2550 60  0000 C CNN
@@
 $EndComp
 $Comp
-L GND #PWR011
+L GND #PWR010
 U 1 1 528AE493
 P 1700 3200
-F 0 "#PWR011" H 1700 3200 30  0001 C CNN
+F 0 "#PWR010" H 1700 3200 30  0001 C CNN
 F 1 "GND" H 1700 3130 30  0001 C CNN
 F 2 "" H 1700 3200 60  0000 C CNN
@@
 	5250 2450 5250 2250
 $Comp
-L +5V #PWR012
+L +5V #PWR011
 U 1 1 528AE608
 P 4900 1250
-F 0 "#PWR012" H 4900 1340 20  0001 C CNN
+F 0 "#PWR011" H 4900 1340 20  0001 C CNN
 F 1 "+5V" H 4900 1340 30  0000 C CNN
 F 2 "" H 4900 1250 60  0000 C CNN
@@
 $EndComp
 $Comp
-L +5V #PWR013
+L +5V #PWR012
 U 1 1 528AE623
 P 5250 1250
-F 0 "#PWR013" H 5250 1340 20  0001 C CNN
+F 0 "#PWR012" H 5250 1340 20  0001 C CNN
 F 1 "+5V" H 5250 1340 30  0000 C CNN
 F 2 "" H 5250 1250 60  0000 C CNN
@@
 	6650 4200 7000 4200
 $Comp
-L GND #PWR014
+L GND #PWR013
 U 1 1 528AE866
 P 6650 4500
-F 0 "#PWR014" H 6650 4500 30  0001 C CNN
+F 0 "#PWR013" H 6650 4500 30  0001 C CNN
 F 1 "GND" H 6650 4430 30  0001 C CNN
 F 2 "" H 6650 4500 60  0000 C CNN
@@
 	6650 4400 7000 4400
 $Comp
-L CONN_6 P4
+L CONN_6 P3
 U 1 1 528AE8AE
 P 6200 4500
-F 0 "P4" V 6150 4500 60  0000 C CNN
-F 1 "CONN_6" V 6250 4500 60  0000 C CNN
+F 0 "P3" V 6150 4500 60  0000 C CNN
+F 1 "FTDI" V 6250 4500 60  0000 C CNN
 F 2 "" H 6200 4500 60  0000 C CNN
 F 3 "" H 6200 4500 60  0000 C CNN
@@
 	5700 4750 5850 4750
 $Comp
-L +5V #PWR015
+L +5V #PWR014
 U 1 1 528AE8BC
 P 5400 4400
-F 0 "#PWR015" H 5400 4490 20  0001 C CNN
+F 0 "#PWR014" H 5400 4490 20  0001 C CNN
 F 1 "+5V" H 5400 4490 30  0000 C CNN
 F 2 "" H 5400 4400 60  0000 C CNN
@@
 	5400 4450 5400 4400
 $Comp
-L GND #PWR016
+L GND #PWR015
 U 1 1 528AE8C4
 P 5650 4100
-F 0 "#PWR016" H 5650 4100 30  0001 C CNN
+F 0 "#PWR015" H 5650 4100 30  0001 C CNN
 F 1 "GND" H 5650 4030 30  0001 C CNN
 F 2 "" H 5650 4100 60  0000 C CNN
@@
 Text Notes 5750 1200 0    60   ~ 0
 RS485
-$Comp
-L CONN_6 P3
-U 1 1 528AE96C
-P 5050 4500
-F 0 "P3" V 5000 4500 60  0000 C CNN
-F 1 "CONN_6" V 5100 4500 60  0000 C CNN
-F 2 "" H 5050 4500 60  0000 C CNN
-F 3 "" H 5050 4500 60  0000 C CNN
-	1    5050 4500
-	1    0    0    -1
-$EndComp
 Wire Notes Line
 	5450 3600 5450 1100
@@
 Text Notes 1000 1250 0    60   ~ 0
 FTDI
+Wire Wire Line
+	3050 3450 3650 3450
+Connection ~ 3500 3450
+$Comp
+L GND #PWR016
+U 1 1 528AF7F5
+P 3500 3550
+F 0 "#PWR016" H 3500 3550 30  0001 C CNN
+F 1 "GND" H 3500 3480 30  0001 C CNN
+F 2 "" H 3500 3550 60  0000 C CNN
+F 3 "" H 3500 3550 60  0000 C CNN
+	1    3500 3550
+	1    0    0    -1
+$EndComp
+Wire Wire Line
+	3500 3450 3500 3550
+$Comp
+L LED LED3
+U 1 1 528AFAFD
+P 6800 1500
+F 0 "LED3" H 6800 1600 50  0000 C CNN
+F 1 "PWR" H 6800 1400 50  0000 C CNN
+F 2 "~" H 6800 1500 60  0000 C CNN
+F 3 "~" H 6800 1500 60  0000 C CNN
+	1    6800 1500
+	1    0    0    -1
+$EndComp
+$Comp
+L R R4
+U 1 1 528AFB04
+P 6250 1500
+F 0 "R4" V 6330 1500 40  0000 C CNN
+F 1 "1k" V 6257 1501 40  0000 C CNN
+F 2 "~" V 6180 1500 30  0000 C CNN
+F 3 "~" H 6250 1500 30  0000 C CNN
+	1    6250 1500
+	0    -1   -1   0
+$EndComp
+$Comp
+L +5V #PWR017
+U 1 1 528AFB0A
+P 5900 1400
+F 0 "#PWR017" H 5900 1490 20  0001 C CNN
+F 1 "+5V" H 5900 1490 30  0000 C CNN
+F 2 "" H 5900 1400 60  0000 C CNN
+F 3 "" H 5900 1400 60  0000 C CNN
+	1    5900 1400
+	1    0    0    -1
+$EndComp
+Wire Wire Line
+	5900 1400 5900 1500
+Wire Wire Line
+	5900 1500 6000 1500
+$Comp
+L GND #PWR018
+U 1 1 528AFBE5
+P 7150 1600
+F 0 "#PWR018" H 7150 1600 30  0001 C CNN
+F 1 "GND" H 7150 1530 30  0001 C CNN
+F 2 "" H 7150 1600 60  0000 C CNN
+F 3 "" H 7150 1600 60  0000 C CNN
+	1    7150 1600
+	1    0    0    -1
+$EndComp
+Wire Wire Line
+	7000 1500 7150 1500
+Wire Wire Line
+	7150 1500 7150 1600
+Wire Wire Line
+	6500 1500 6600 1500
 $EndSCHEMATC

Commit message: Filled board, added logos text
Parts:
- C1: value C -> 47u
- P5: value CONN_2 -> PWR
- R1, R2: value R -> 1k
Changed lines of the file:
@@
 Sheet 1 1
 Title "RS485 to USB Converter with RJ45"
-Date "19 nov 2013"
+Date "20 nov 2013"
 Rev "1"
 Comp "Visgence Inc"
@@
 P 1700 2850
 F 0 "C1" H 1700 2950 40  0000 L CNN
-F 1 "C" H 1706 2765 40  0000 L CNN
+F 1 "47u" H 1706 2765 40  0000 L CNN
 F 2 "~" H 1738 2700 30  0000 C CNN
 F 3 "~" H 1700 2850 60  0000 C CNN
@@
 P 4900 1550
 F 0 "R1" V 4980 1550 40  0000 C CNN
-F 1 "R" V 4907 1551 40  0000 C CNN
+F 1 "1k" V 4907 1551 40  0000 C CNN
 F 2 "~" V 4830 1550 30  0000 C CNN
 F 3 "~" H 4900 1550 30  0000 C CNN
@@
 P 5250 1550
 F 0 "R2" V 5330 1550 40  0000 C CNN
-F 1 "R" V 5257 1551 40  0000 C CNN
+F 1 "1k" V 5257 1551 40  0000 C CNN
 F 2 "~" V 5180 1550 30  0000 C CNN
 F 3 "~" H 5250 1550 30  0000 C CNN
@@
 P 7350 4300
 F 0 "P5" V 7300 4300 40  0000 C CNN
-F 1 "CONN_2" V 7400 4300 40  0000 C CNN
+F 1 "PWR" V 7400 4300 40  0000 C CNN
 F 2 "" H 7350 4300 60  0000 C CNN
 F 3 "" H 7350 4300 60  0000 C CNN
