File: rs485-usb.kicad_pcb (KiCad board)
At the start: 2 copper layers, 67.3 x 20.3 mm, 13 parts, among them J1 RJ45, P1 USBMICRO, P2 FTDI, P3 FTDI, P5 CONN_2, U1 FT232RL, U2 MAX488

Commit message: Filled board, added logos text
Parts:
- added G***: LOGO, LOGO, B.Cu at (39.9, 34.8)
- added G2: LOGO, OSHW_LOGO, B.Cu at (66.5, 32.3)
- added LED3: PWR, LED-0603, F.Cu at (67.9, 27.9)
- added R4: 1k, SM0603, F.Cu at (64.1, 27.9)
- C1: value C -> 47u
- P5: value CONN_2 -> PWR
- R1, R2: value R -> 1k
Connections:
- J1 pad : (no net) -> GND
- P1 pad : (no net) -> GND
Routing:
- net +5V: track 103.9 -> 107.6 mm
- net N-000021: track 0.00 -> 2.30 mm
- added copper zone on B.Cu, net GND
- added copper zone on F.Cu, net GND
Other:
- board text added: "+"
- board text added: "-"
- board text added: "2013 Visgence Inc."
- board text added: "5V"
- board text added: "CTS"
- board text added: "DTR"
- board text added: "GND"
- board text added: "RX"
- board text added: "TX"
- board text added: "USB to full duplex RS485"

Commit message: Added gerber rules
Parts:
- moved G*** 0.80 mm to (39.1, 34.5)
Changed lines of the file:
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@@
     (visible_elements 7FFFFFFF)
     (pcbplotparams
-      (layerselection 3178497)
+      (layerselection 284196865)
       (usegerberextensions true)
-      (excludeedgelayer true)
+      (excludeedgelayer false)
       (linewidth 0.150000)
       (plotframeref false)
@@
       (plotinvisibletext false)
       (padsonsilk false)
-      (subtractmaskfromsilk false)
+      (subtractmaskfromsilk true)
       (outputformat 1)
       (mirror false)
-      (drillshape 1)
+      (drillshape 0)
       (scaleselection 1)
-      (outputdirectory ""))
+      (outputdirectory gerber/))
   )
   (net 0 "")
@@
   )
   (module LOGO (layer B.Cu)
-    (at 39.878 34.798)
+    (at 39.116 34.544)
     (fp_text reference G*** (at 0 -7.19582) (layer B.SilkS) hide
       (effects (font (size 1.524 1.524) (thickness 0.3048)) (justify mirror))
@@
     (effects (font (size 0.6 0.6) (thickness 0.1016)))
   )
-  (gr_text "USB to full duplex RS485" (at 64.77 42.672) (layer B.SilkS)
+  (gr_text "USB to full duplex RS485" (at 66.548 39.624) (layer B.SilkS)
     (effects (font (size 0.889 0.889) (thickness 0.22225)) (justify mirror))
   )
-  (gr_text "2013 Visgence Inc." (at 66.04 40.894) (layer B.SilkS)
+  (gr_text "2013 Visgence Inc." (at 66.294 38.1) (layer B.SilkS)
     (effects (font (size 0.889 0.889) (thickness 0.22225)) (justify mirror))
   )
-  (gr_text "USB to full duplex RS485" (at 38.862 42.672) (layer B.SilkS)
+  (gr_text "USB to full duplex RS485" (at 44.196 44.45) (layer B.SilkS)
     (effects (font (size 0.889 0.889) (thickness 0.22225)) (justify mirror))
   )
-  (gr_text "2013 Visgence Inc." (at 38.862 41.148) (layer B.SilkS)
+  (gr_text "2013 Visgence Inc." (at 42.418 42.926) (layer B.SilkS)
     (effects (font (size 0.889 0.889) (thickness 0.22225)) (justify mirror))
   )
